File: hardware/kicad-slave-pcb/espir_slave_pcb.kicad_pcb (KiCad board)
At the start: 4 copper layers, 66 x 47.1 mm, 38 parts, among them Q2 AO3400A, Q4 AO3401A, SW1 RESET, SW2 BOOT, SW3 SS12D07VG6, U2 IR333C, U3 IR333C, U5 ESP32-C6-MINI-1, U6 AP2112K-3.3, U7 LiPo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

Commit message: hardware: pour GND planes before routing (no redundant GND traces)
Root cause of the redundant GND traces: the pipeline routed first, so
Freerouting filled GND with traces (119 here) that the pour then made
pointless. A filled GND zone exports to the Specctra DSN as (plane GND ...)
per layer, so pouring the planes BEFORE routing makes Freerouting treat GND as
already-connected and route only the signal nets (adding just the pad-to-plane
vias GND needs).

- pour_gnd.py: add a `planes-only` mode (fill, no stitching) for the pre-route
  pour; the full mode (re-fill + stitch) still runs after routing.
- build.sh: reorder to place -> pour planes-only -> route -> re-fill + stitch -> DRC.
- route.sh / README: document the plane-export behaviour and new order.
- espir_slave_pcb.kicad_pcb: apply the same cleanup to the existing board —
  removed 61 redundant open-area GND traces (~115 mm; 119 -> 58 segments, all
  inner-layer GND traces gone). Kept the traces knitting U5's fenced-in module
  GND pins (the pour can't reach between them). DRC: 0 unconnected, 0 electrical
  violations.
Routing:
- net GND: track 226.1 -> 111.0 mm
